Commit message: Added mouse w/o sensors

File: mouse_gazebo/models/box.xacro (robot description, xacro)
@@ -2,9 +2,9 @@
 <robot name="box" xmlns:xacro="http://www.ros.org/wiki/xacro">
 <!-- TODO adjust parameters -->
-	<xacro:property name="len" value="0.3"/>
+	<xacro:property name="len" value="0.25"/>
 	<xacro:property name="mass" value="1"/>
 	<link name="base_link">
 		<visual>
-			<origin xyz="0 0 0" rpy="0 0 0"/>
+			<origin xyz="0 0 ${len/2}" rpy="0 0 0"/>
 			<geometry>
 				<box size="${len} ${len} ${len}"/>
@@ -12,5 +12,5 @@
 		</visual>
 		<collision>
-			<origin xyz="0 0 0" rpy="0 0 0"/>
+			<origin xyz="0 0 ${len/2}" rpy="0 0 0"/>
 			<geometry>
 				<box size="${len} ${len} ${len}"/>
@@ -18,5 +18,5 @@
 		</collision>
 		<inertial>
-			<origin xyz="0 0 0" rpy="0 0 0"/>
+			<origin xyz="0 0 ${len/2}" rpy="0 0 0"/>
 			<mass value="${mass}"/>
 			<inertia
