Commit message: Spawn 4 mice

File: mouse_description/urdf/mouse.xacro (robot description, xacro)
@@ -36,4 +36,5 @@
 		</gazebo>
 	</link>
+	<!-- Actuation -->
 	<link name="left_wheel">
 		<visual>
@@ -58,6 +59,6 @@
 		</inertial>
 		<gazebo reference="left_wheel">
-			<mu1>0.5</mu1>
-			<mu2>0.5</mu2>
+			<mu1>1.0</mu1>
+			<mu2>1.0</mu2>
 			<kp>1000000.0</kp>
 			<kd>100.0</kd>
@@ -88,6 +89,6 @@
 		</inertial>
 		<gazebo reference="right_wheel">
-			<mu1>0.5</mu1>
-			<mu2>0.5</mu2>
+			<mu1>1.0</mu1>
+			<mu2>1.0</mu2>
 			<kp>1000000.0</kp>
 			<kd>100.0</kd>
@@ -112,5 +113,11 @@
 		<limit effort="${wheel_torque}" velocity="${wheel_veloc}"/>
 	</joint>
+	<!-- Sensors -->
 	<!-- Gazebo Sensors -->
+	<!-- TODO add IR sensors -->
+	<!-- TODO add IMU sensor -->
+	<!-- TODO add mouse sensor -->
+	<!-- TODO add front color sensor -->
+	<!-- TODO add GPS sensor -->
 	<!-- Gazebo Actuation -->
 	<gazebo>
@@ -118,5 +125,5 @@
 			<rosDebugLevel>0</rosDebugLevel>
 			<alwaysOn>true</alwaysOn>
-			<updateRate>60</updateRate>
+			<updateRate>100</updateRate>
 			<leftJoint>right_mot</leftJoint>
 			<rightJoint>left_mot</rightJoint>
@@ -127,4 +134,5 @@
 			<commandTopic>$(arg name)/cmd_vel</commandTopic>
 			<odometryTopic>$(arg name)/odom</odometryTopic>
+			<!-- world == perfect positioning -->
 			<odometrySource>world</odometrySource>
 			<odometryFrame>$(arg name)/odom</odometryFrame>

File: mouse_gazebo/models/box.xacro (robot description, xacro)
@@ -3,5 +3,5 @@
 <!-- TODO adjust parameters -->
 	<xacro:property name="len" value="0.25"/>
-	<xacro:property name="mass" value="1"/>
+	<xacro:property name="mass" value="0.5"/>
 	<link name="base_link">
 		<visual>

Commit message: Added IR sensors

File: mouse_description/urdf/mouse.xacro (robot description, xacro)
@@ -117,5 +117,5 @@
 			<rosDebugLevel>0</rosDebugLevel>
 			<alwaysOn>true</alwaysOn>
-			<updateRate>100</updateRate>
+			<updateRate>120</updateRate>
 			<leftJoint>right_mot</leftJoint>
 			<rightJoint>left_mot</rightJoint>
@@ -137,6 +137,202 @@
 	</gazebo>
 	<!-- Sensors -->
-	<!-- Gazebo Sensors -->
-	<!-- TODO add IR sensors -->
+	<!-- IR sensors -->
+	<link name="left_ir">
+		<visual>
+			<geometry>
+				<box size="0.001 0.001 0.001"/>
+			</geometry>
+		</visual>
+		<collision>
+			<geometry>
+				<box size="0.001 0.001 0.001"/>
+			</geometry>
+		</collision>
+		<inertial>
+			<mass value="1e-6"/>
+			<inertia
+        		ixx="1e-7" ixy="0.0" ixz="0.0"
+        		iyy="1e-7" iyz="0.0"
+        		izz="1e-7"/>
+		</inertial>
+	</link>
+	<link name="right_ir">
+		<visual>
+			<geometry>
+				<box size="0.001 0.001 0.001"/>
+			</geometry>
+		</visual>
+		<collision>
+			<geometry>
+				<box size="0.001 0.001 0.001"/>
+			</geometry>
+		</collision>
+		<inertial>
+			<mass value="1e-6"/>
+			<inertia
+        		ixx="1e-7" ixy="0.0" ixz="0.0"
+        		iyy="1e-7" iyz="0.0"
+        		izz="1e-7"/>
+		</inertial>
+	</link>
+	<link name="left_front_ir">
+		<visual>
+			<geometry>
+				<box size="0.001 0.001 0.001"/>
+			</geometry>
+		</visual>
+		<collision>
+			<geometry>
+				<box size="0.001 0.001 0.001"/>
+			</geometry>
+		</collision>
+		<inertial>
+			<mass value="1e-6"/>
+			<inertia
+        		ixx="1e-7" ixy="0.0" ixz="0.0"
+        		iyy="1e-7" iyz="0.0"
+        		izz="1e-7"/>
+		</inertial>
+	</link>
+	<link name="right_front_ir">
+		<visual>
+			<geometry>
+				<box size="0.001 0.001 0.001"/>
+			</geometry>
+		</visual>
+		<collision>
+			<geometry>
+				<box size="0.001 0.001 0.001"/>
+			</geometry>
+		</collision>
+		<inertial>
+			<mass value="1e-6"/>
+			<inertia
+        		ixx="1e-7" ixy="0.0" ixz="0.0"
+        		iyy="1e-7" iyz="0.0"
+        		izz="1e-7"/>
+		</inertial>
+	</link>
+	<joint name="left_ir_mnt" type="fixed">
+		<origin xyz="-0.0256 0.0207 0.013" rpy="0 0 1.5708"/>
+		<parent link="base_link"/>
+		<child link="left_ir"/>
+	</joint>
+	<joint name="right_ir_mnt" type="fixed">
+		<origin xyz="0.0256 0.0207 0.013" rpy="0 0 1.5708"/>
+		<parent link="base_link"/>
+		<child link="right_ir"/>
+	</joint>
+	<joint name="left_front_ir_mnt" type="fixed">
+		<origin xyz="-0.009152 0.032074 0.013" rpy="0 0 2.4347"/>
+		<parent link="base_link"/>
+		<child link="left_front_ir"/>
+	</joint>
+	<joint name="right_front_ir_mnt" type="fixed">
+		<origin xyz="0.009152 0.032074 0.013" rpy="0 0 0.70686"/>
+		<parent link="base_link"/>
+		<child link="right_front_ir"/>
+	</joint>
+	<gazebo reference="left_ir">
+		<sensor type="ray" name="left_ir_sens">
+			<pose>0 0 0 0 0 0</pose>
+			<visualize>true</visualize>
+			<update_rate>30</update_rate>
+			<ray>
+				<scan>
+					<horizontal>
+						<samples>3</samples>
+						<resolution>1</resolution>
+						<min_angle>-0.01</min_angle>
+						<max_angle>0.01</max_angle>
+					</horizontal>
+				</scan>
+				<range>
+					<min>0.01</min>
+					<max>0.5</max>
+					<resolution>0.001</resolution>
+				</range>
+			</ray>
+			<plugin filename="libgazebo_ros_laser.so" name="gazebo_ros_gpu_laser">
+				<topicName>left_ir</topicName>
+				<frameName>left_ir</frameName>
+			</plugin>
+		</sensor>
+	</gazebo>
+	<gazebo reference="right_ir">
+		<sensor type="ray" name="right_ir_sens">
+			<pose>0 0 0 0 0 0</pose>
+			<visualize>true</visualize>
+			<update_rate>30</update_rate>
+			<ray>
+				<scan>
+					<horizontal>
+						<samples>3</samples>
+						<min_angle>-0.01</min_angle>
+						<max_angle>0.01</max_angle>
+					</horizontal>
+				</scan>
+				<range>
+					<min>0.01</min>
+					<max>0.5</max>
+					<resolution>0.001</resolution>
+				</range>
+			</ray>
+			<plugin filename="libgazebo_ros_laser.so" name="gazebo_ros_gpu_laser">
+				<topicName>right_ir</topicName>
+				<frameName>right_ir</frameName>
+			</plugin>
+		</sensor>
+	</gazebo>
+	<gazebo reference="left_front_ir">
+		<sensor type="ray" name="left_front_ir_sens">
+			<pose>0 0 0 0 0 0</pose>
+			<visualize>true</visualize>
+			<update_rate>30</update_rate>
+			<ray>
+				<scan>
+					<horizontal>
+						<samples>3</samples>
+						<min_angle>-0.01</min_angle>
+						<max_angle>0.01</max_angle>
+					</horizontal>
+				</scan>
+				<range>
+					<min>0.01</min>
+					<max>0.5</max>
+					<resolution>0.001</resolution>
+				</range>
+			</ray>
+			<plugin filename="libgazebo_ros_laser.so" name="gazebo_ros_gpu_laser">
+				<topicName>left_front_ir</topicName>
+				<frameName>left_front_ir</frameName>
+			</plugin>
+		</sensor>
+	</gazebo>
+	<gazebo reference="right_front_ir">
+		<sensor type="ray" name="right_front_ir_sens">
+			<pose>0 0 0 0 0 0</pose>
+			<visualize>true</visualize>
+			<update_rate>30</update_rate>
+			<ray>
+				<scan>
+					<horizontal>
+						<samples>3</samples>
+						<min_angle>-0.01</min_angle>
+						<max_angle>0.01</max_angle>
+					</horizontal>
+				</scan>
+				<range>
+					<min>0.01</min>
+					<max>0.5</max>
+					<resolution>0.001</resolution>
+				</range>
+			</ray>
+			<plugin filename="libgazebo_ros_laser.so" name="gazebo_ros_gpu_laser">
+				<topicName>right_front_ir</topicName>
+				<frameName>right_front_ir</frameName>
+			</plugin>
+		</sensor>
+	</gazebo>
 	<!-- TODO add IMU sensor -->
 	<!-- TODO add mouse sensor -->

Commit message: Added bumper sensors

File: mouse_description/urdf/mouse.xacro (robot description, xacro)
@@ -7,11 +7,9 @@
 	<link name="base_link">
 		<visual>
-			<origin xyz="0 0 0" rpy="0 0 0"/>
 			<geometry>
 				<mesh filename="package://mouse_description/meshes/mouse_base.dae" scale="1 1 1"/>
 			</geometry>
 		</visual>
-		<collision>
-			<origin xyz="0 0 0" rpy="0 0 0"/>
+		<collision name="base_link_collision">
 			<geometry>
 				<mesh filename="package://mouse_description/meshes/mouse_base.dae" scale="1 1 1"/>
@@ -31,5 +29,5 @@
 			<kp>1000000.0</kp>
 			<kd>100.0</kd>
-			<minDepth>0.001</minDepth>
+			<minDepth>0.0001</minDepth>
 			<maxVel>1.0</maxVel>
 		</gazebo>
@@ -38,11 +36,9 @@
 	<link name="left_wheel">
 		<visual>
-			<origin xyz="0 0 0" rpy="0 0 0"/>
 			<geometry>
 				<mesh filename="package://mouse_description/meshes/mouse_wheel.dae" scale="1 1 1"/>
 			</geometry>
 		</visual>
-		<collision>
-			<origin xyz="0 0 0" rpy="0 0 0"/>
+		<collision name="left_wheel_collision">
 			<geometry>
 				<mesh filename="package://mouse_description/meshes/mouse_wheel.dae" scale="1 1 1"/>
@@ -50,5 +46,4 @@
 		</collision>
 		<inertial>
-			<origin xyz="0 0 0" rpy="0 0 0"/>
 			<mass value="0.015"/>
 			<inertia
@@ -57,22 +52,12 @@
         		izz="1.146e-6"/>
 		</inertial>
-		<gazebo reference="left_wheel">
-			<mu1>1.0</mu1>
-			<mu2>1.0</mu2>
-			<kp>1000000.0</kp>
-			<kd>100.0</kd>
-			<minDepth>0.001</minDepth>
-			<maxVel>1.0</maxVel>
-		</gazebo>
 	</link>
 	<link name="right_wheel">
 		<visual>
-			<origin xyz="0 0 0" rpy="0 0 0"/>
 			<geometry>
 				<mesh filename="package://mouse_description/meshes/mouse_wheel.dae" scale="1 1 1"/>
 			</geometry>
 		</visual>
-		<collision>
-			<origin xyz="0 0 0" rpy="0 0 0"/>
+		<collision name="right_wheel_collision">
 			<geometry>
 				<mesh filename="package://mouse_description/meshes/mouse_wheel.dae" scale="1 1 1"/>
@@ -80,5 +65,4 @@
 		</collision>
 		<inertial>
-			<origin xyz="0 0 0" rpy="0 0 0"/>
 			<mass value="0.015"/>
 			<inertia
@@ -87,12 +71,4 @@
         		izz="1.146e-6"/>
 		</inertial>
-		<gazebo reference="right_wheel">
-			<mu1>1.0</mu1>
-			<mu2>1.0</mu2>
-			<kp>1000000.0</kp>
-			<kd>100.0</kd>
-			<minDepth>0.001</minDepth>
-			<maxVel>1.0</maxVel>
-		</gazebo>
 	</link>
 	<joint name="left_mot" type="continuous">
@@ -101,5 +77,5 @@
 		<origin xyz="${wheel_sep/2} 0 ${wheel_dia/2}" rpy="0 0 0"/>
 		<axis xyz="-1 0 0"/>
-		<dynamics friction="0.001"/>
+		<dynamics friction="0.01"/>
 		<limit effort="${wheel_torque}" velocity="${wheel_veloc}"/>
 	</joint>
@@ -109,7 +85,25 @@
 		<origin xyz="${-wheel_sep/2} 0 ${wheel_dia/2}" rpy="0 0 0"/>
 		<axis xyz="-1 0 0"/>
-		<dynamics friction="0.001"/>
+		<dynamics friction="0.01"/>
 		<limit effort="${wheel_torque}" velocity="${wheel_veloc}"/>
 	</joint>
+	<gazebo reference="left_wheel">
+		<mu1>1.0</mu1>
+		<mu2>1.0</mu2>
+		<kp>1000000.0</kp>
+		<kd>100.0</kd>
+		<minDepth>0.0001</minDepth>
+		<maxVel>1.0</maxVel>
+		<material>Gazebo/Black</material>
+	</gazebo>
+	<gazebo reference="right_wheel">
+		<mu1>1.0</mu1>
+		<mu2>1.0</mu2>
+		<kp>1000000.0</kp>
+		<kd>100.0</kd>
+		<minDepth>0.0001</minDepth>
+		<maxVel>1.0</maxVel>
+		<material>Gazebo/Black</material>
+	</gazebo>
 	<!-- Gazebo Actuation -->
 	<gazebo>
@@ -137,205 +131,191 @@
 	</gazebo>
 	<!-- Sensors -->
-	<!-- IR sensors -->
-	<link name="left_ir">
-		<visual>
-			<geometry>
-				<box size="0.001 0.001 0.001"/>
-			</geometry>
-		</visual>
-		<collision>
-			<geometry>
-				<box size="0.001 0.001 0.001"/>
-			</geometry>
-		</collision>
-		<inertial>
-			<mass value="1e-6"/>
-			<inertia
-        		ixx="1e-7" ixy="0.0" ixz="0.0"
-        		iyy="1e-7" iyz="0.0"
-        		izz="1e-7"/>
-		</inertial>
-	</link>
-	<link name="right_ir">
-		<visual>
-			<geometry>
-				<box size="0.001 0.001 0.001"/>
-			</geometry>
-		</visual>
-		<collision>
-			<geometry>
-				<box size="0.001 0.001 0.001"/>
-			</geometry>
-		</collision>
-		<inertial>
-			<mass value="1e-6"/>
-			<inertia
-        		ixx="1e-7" ixy="0.0" ixz="0.0"
-        		iyy="1e-7" iyz="0.0"
-        		izz="1e-7"/>
-		</inertial>
-	</link>
-	<link name="left_front_ir">
-		<visual>
-			<geometry>
-				<box size="0.001 0.001 0.001"/>
-			</geometry>
-		</visual>
-		<collision>
-			<geometry>
-				<box size="0.001 0.001 0.001"/>
-			</geometry>
-		</collision>
-		<inertial>
-			<mass value="1e-6"/>
-			<inertia
-        		ixx="1e-7" ixy="0.0" ixz="0.0"
-        		iyy="1e-7" iyz="0.0"
-        		izz="1e-7"/>
-		</inertial>
-	</link>
-	<link name="right_front_ir">
-		<visual>
-			<geometry>
-				<box size="0.001 0.001 0.001"/>
-			</geometry>
-		</visual>
-		<collision>
-			<geometry>
-				<box size="0.001 0.001 0.001"/>
-			</geometry>
-		</collision>
-		<inertial>
-			<mass value="1e-6"/>
-			<inertia
-        		ixx="1e-7" ixy="0.0" ixz="0.0"
-        		iyy="1e-7" iyz="0.0"
-        		izz="1e-7"/>
-		</inertial>
-	</link>
-	<joint name="left_ir_mnt" type="fixed">
-		<origin xyz="-0.0256 0.0207 0.013" rpy="0 0 1.5708"/>
-		<parent link="base_link"/>
-		<child link="left_ir"/>
-	</joint>
-	<joint name="right_ir_mnt" type="fixed">
-		<origin xyz="0.0256 0.0207 0.013" rpy="0 0 1.5708"/>
-		<parent link="base_link"/>
-		<child link="right_ir"/>
-	</joint>
-	<joint name="left_front_ir_mnt" type="fixed">
-		<origin xyz="-0.009152 0.032074 0.013" rpy="0 0 2.4347"/>
-		<parent link="base_link"/>
-		<child link="left_front_ir"/>
-	</joint>
-	<joint name="right_front_ir_mnt" type="fixed">
-		<origin xyz="0.009152 0.032074 0.013" rpy="0 0 0.70686"/>
-		<parent link="base_link"/>
-		<child link="right_front_ir"/>
-	</joint>
-	<gazebo reference="left_ir">
-		<sensor type="ray" name="left_ir_sens">
-			<pose>0 0 0 0 0 0</pose>
-			<visualize>true</visualize>
-			<update_rate>30</update_rate>
-			<ray>
-				<scan>
-					<horizontal>
-						<samples>3</samples>
-						<resolution>1</resolution>
-						<min_angle>-0.01</min_angle>
-						<max_angle>0.01</max_angle>
-					</horizontal>
-				</scan>
-				<range>
-					<min>0.01</min>
-					<max>0.5</max>
-					<resolution>0.001</resolution>
-				</range>
-			</ray>
-			<plugin filename="libgazebo_ros_laser.so" name="gazebo_ros_gpu_laser">
-				<topicName>left_ir</topicName>
-				<frameName>left_ir</frameName>
+	<!-- TODO add front color sensor -->
+	<!-- Bumper sensor -->
+	<link name="left_bump">
+		<visual>
+			<geometry>
+				<sphere radius="0.005"/>
+			</geometry>
+		</visual>
+		<collision name="left_bump_collision">
+			<geometry>
+				<sphere radius="0.005"/>
+			</geometry>
+		</collision>
+		<inertial>
+			<mass value="1e-5"/>
+			<inertia
+        		ixx="1e-6" ixy="0.0" ixz="0.0"
+        		iyy="1e-6" iyz="0.0"
+        		izz="1e-6"/>
+		</inertial>
+	</link>
+	<link name="right_bump">
+		<visual>
+			<geometry>
+				<sphere radius="0.005"/>
+			</geometry>
+		</visual>
+		<collision name="right_bump_collision">
+			<geometry>
+				<sphere radius="0.005"/>
+			</geometry>
+		</collision>
+		<inertial>
+			<mass value="1e-5"/>
+			<inertia
+        		ixx="1e-6" ixy="0.0" ixz="0.0"
+        		iyy="1e-6" iyz="0.0"
+        		izz="1e-6"/>
+		</inertial>
+	</link>
+	<link name="left_front_bump">
+		<visual>
+			<geometry>
+				<sphere radius="0.005"/>
+			</geometry>
+		</visual>
+		<collision name="left_front_bump_collision">
+			<geometry>
+				<sphere radius="0.005"/>
+			</geometry>
+		</collision>
+		<inertial>
+			<mass value="1e-5"/>
+			<inertia
+        		ixx="1e-6" ixy="0.0" ixz="0.0"
+        		iyy="1e-6" iyz="0.0"
+        		izz="1e-6"/>
+		</inertial>
+	</link>
+	<link name="right_front_bump">
+		<visual>
+			<geometry>
+				<sphere radius="0.005"/>
+			</geometry>
+		</visual>
+		<collision name="right_front_bump_collision">
+			<geometry>
+				<sphere radius="0.005"/>
+			</geometry>
+		</collision>
+		<inertial>
+			<mass value="1e-5"/>
+			<inertia
+        		ixx="1e-6" ixy="0.0" ixz="0.0"
+        		iyy="1e-6" iyz="0.0"
+        		izz="1e-6"/>
+		</inertial>
+	</link>
+	<joint name="left_bump_mnt" type="fixed">
+		<origin xyz="-0.0256 0.0207 0.013" rpy="0 0 0"/>
+		<parent link="base_link"/>
+		<child link="left_bump"/>
+	</joint>
+	<joint name="right_bump_mnt" type="fixed">
+		<origin xyz="0.0256 0.0207 0.013" rpy="0 0 0"/>
+		<parent link="base_link"/>
+		<child link="right_bump"/>
+	</joint>
+	<joint name="left_front_bump_mnt" type="fixed">
+		<origin xyz="-0.009152 0.032074 0.013" rpy="0 0 0"/>
+		<parent link="base_link"/>
+		<child link="left_front_bump"/>
+	</joint>
+	<joint name="right_front_bump_mnt" type="fixed">
+		<origin xyz="0.009152 0.032074 0.013" rpy="0 0 0"/>
+		<parent link="base_link"/>
+		<child link="right_front_bump"/>
+	</joint>
+	<gazebo reference="left_bump_mnt">
+		<preserveFixedJoint>true</preserveFixedJoint>
+	</gazebo>
+	<gazebo reference="right_bump_mnt">
+		<preserveFixedJoint>true</preserveFixedJoint>
+	</gazebo>
+	<gazebo reference="left_front_bump_mnt">
+		<preserveFixedJoint>true</preserveFixedJoint>
+	</gazebo>
+	<gazebo reference="right_front_bump_mnt">
+		<preserveFixedJoint>true</preserveFixedJoint>
+	</gazebo>
+	<gazebo reference="left_bump">
+		<mu1>1.0</mu1>
+		<mu2>1.0</mu2>
+		<kp>1000000.0</kp>
+		<kd>100.0</kd>
+		<minDepth>0.0001</minDepth>
+		<maxVel>1.0</maxVel>
+		<material>Gazebo/Blue</material>
+		<sensor name="left_bump" type="contact">
+			<updateRate>24</updateRate>
+			<contact>
+				<collision>left_bump_collision_collision</collision>
+			</contact>
+			<plugin name="gazebo_ros_bumper" filename="libgazebo_ros_bumper.so">
+				<bumperTopicName>bumper</bumperTopicName>
+				<frameName>left_bump</frameName>
 			</plugin>
 		</sensor>
 	</gazebo>
-	<gazebo reference="right_ir">
-		<sensor type="ray" name="right_ir_sens">
-			<pose>0 0 0 0 0 0</pose>
-			<visualize>true</visualize>
-			<update_rate>30</update_rate>
-			<ray>
-				<scan>
-					<horizontal>
-						<samples>3</samples>
-						<min_angle>-0.01</min_angle>
-						<max_angle>0.01</max_angle>
-					</horizontal>
-				</scan>
-				<range>
-					<min>0.01</min>
-					<max>0.5</max>
-					<resolution>0.001</resolution>
-				</range>
-			</ray>
-			<plugin filename="libgazebo_ros_laser.so" name="gazebo_ros_gpu_laser">
-				<topicName>right_ir</topicName>
-				<frameName>right_ir</frameName>
+	<gazebo reference="right_bump">
+		<mu1>1.0</mu1>
+		<mu2>1.0</mu2>
+		<kp>1000000.0</kp>
+		<kd>100.0</kd>
+		<minDepth>0.0001</minDepth>
+		<maxVel>1.0</maxVel>
+		<material>Gazebo/Blue</material>
+		<sensor name="right_bump" type="contact">
+			<updateRate>24</updateRate>
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
Commit message: Added camera sensor

File: mouse_description/urdf/mouse.xacro (robot description, xacro)
@@ -131,5 +131,53 @@
 	</gazebo>
 	<!-- Sensors -->
-	<!-- TODO add front color sensor -->
+	<!-- Color Sensor (Camera) -->
+	<link name="front_cam">
+		<visual>
+			<geometry>
+				<box size="0.008 0.008 0.008"/>
+			</geometry>
+		</visual>
+		<collision name="front_cam_collision">
+			<geometry>
+				<box size="0.008 0.008 0.008"/>
+			</geometry>
+		</collision>
+		<inertial>
+			<mass value="1e-5"/>
+			<inertia
+        		ixx="1e-6" ixy="0.0" ixz="0.0"
+        		iyy="1e-6" iyz="0.0"
+        		izz="1e-6"/>
+		</inertial>
+	</link>
+	<joint name="front_cam_mnt" type="fixed">
+		<origin xyz="0 0 0.027" rpy="0 0 1.5708"/>
+		<parent link="base_link"/>
+		<child link="front_cam"/>
+	</joint>
+	<gazebo reference="front_cam">
+		<material>Gazebo/Blue</material>
+		<sensor name="front_cam" type="camera">
+			<update_rate>24</update_rate>
+			<camera name="front_cam">
+				<horizontal_fov>2</horizontal_fov>
+				<image>
+					<width>640</width>
+					<height>480</height>
+					<format>R8G8B8</format>
+				</image>
+				<clip>
+					<near>0.001</near>
+					<far>0.5</far>
+				</clip>
+			</camera>
+			<plugin name="gazebo_ros_camera" filename="libgazebo_ros_camera.so">
+				<imageTopicName>image_raw</imageTopicName>
+				<cameraInfoTopicName>camera_info</cameraInfoTopicName>
+				<!-- incorrect TF frame -->
+				<frameName>base</frameName>
+			</plugin>
+		</sensor>
+	</gazebo>
 	<!-- Bumper sensor -->
 	<link name="left_bump">

Commit message: Fixed ghostbox and improved color sensor

File: mouse_description/urdf/mouse.xacro (robot description, xacro)
@@ -152,5 +152,5 @@
 	</link>
 	<joint name="front_cam_mnt" type="fixed">
-		<origin xyz="0 0 0.027" rpy="0 0 1.5708"/>
+		<origin xyz="0 0.0025 0.027" rpy="0 0 1.57079632679"/>
 		<parent link="base_link"/>
 		<child link="front_cam"/>
@@ -161,13 +161,13 @@
 			<update_rate>30</update_rate>
 			<camera name="front_cam">
-				<horizontal_fov>2</horizontal_fov>
+				<horizontal_fov>2.65</horizontal_fov>
 				<image>
 					<width>640</width>
-					<height>480</height>
+					<height>360</height>
 					<format>R8G8B8</format>
 				</image>
 				<clip>
 					<near>0.001</near>
-					<far>0.5</far>
+					<far>0.25</far>
 				</clip>
 			</camera>

File: mouse_gazebo/models/ghostbox.xacro (robot description, xacro)
@@ -11,5 +11,5 @@
 		</visual>
 		<!-- Collision bitmasks not parsed properly currently -->
-		<!-- So here's the janky workaround -->
+		<!-- So here's the janky workaround, actually cleaner -->
 		<inertial>
 			<origin xyz="0 0 ${len/2}" rpy="0 0 0"/>
@@ -22,4 +22,7 @@
 	</link>
 	<gazebo reference="base_link">
+		<visual>
+			<plugin name="invisible" filename="libmouse_gazebo.so"/>
+		</visual>
 		<turnGravityOff>true</turnGravityOff>
 		<material>Gazebo/GreenTransparent</material>
